File: hat_rev8/hat_rev8.kicad_pcb (KiCad board)
At the start: 2 copper layers, 65 x 56 mm, 35 parts, among them J1 RPi 4, J6 DNP-Conn_01x05, J7 DNP-Conn_01x05, SW1 JOYSTICK, T1 BSS138, T2 BSS138, T3 BSS138, U1 SHT40

Commit message: add bling
Other:
- board text added: "APROG V8: 07/26"
- board text removed: "V8: 07/26"
