File: hat_rev8/hat_rev8.kicad_pcb (KiCad board)
At the start: 2 copper layers, 65 x 56 mm, 35 parts, among them J1 RPi 4, J6 DNP-Conn_01x05, J7 DNP-Conn_01x05, SW1 JOYSTICK, T1 BSS138, T2 BSS138, T3 BSS138, U1 SHT40

Commit message: update dual diode to BAT54C
Parts:
- D1, D2, D3, D7, D8: value PMEG2005CT -> BAT54C
Changed lines of the file:
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@@
 			)
 		)
-		(property "Value" "PMEG2005CT"
+		(property "Value" "BAT54C"
 			(at 0 2.5 180)
 			(layer "F.Fab")
@@
 			)
 		)
-		(property "Value" "PMEG2005CT"
+		(property "Value" "BAT54C"
 			(at 0 2.5 0)
 			(layer "F.Fab")
@@
 			)
 		)
-		(property "Value" "PMEG2005CT"
+		(property "Value" "BAT54C"
 			(at 0 2.5 0)
 			(layer "F.Fab")
@@
 			)
 		)
-		(property "Value" "PMEG2005CT"
+		(property "Value" "BAT54C"
 			(at 0 2.5 0)
 			(layer "F.Fab")
@@
 			)
 		)
-		(property "Value" "PMEG2005CT"
+		(property "Value" "BAT54C"
 			(at 0 2.5 0)
 			(layer "F.Fab")
