File: hat_rev8/hat_rev8.kicad_sch (KiCad schematic)
At the start: 31 parts, among them J1 RPi 4, J6 DNP-Conn_01x05, J7 DNP-Conn_01x05, SW1 JOYSTICK, T1 BSS138, T2 BSS138, T3 BSS138, U1 SHT40

Commit message: update dual diode to BAT54C
Parts:
- D1, D2, D3, D7, D8: value PMEG2005CT -> BAT54C
Other:
- note removed: "Replacement part for PMEG2005: PMEG3005 PMEG4005 same diode, slightly higher Vf, higher reverse voltage"
Changed lines of the file:
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@@
 		)
 	)
-	(text "Replacement part for PMEG2005:\nPMEG3005\nPMEG4005\nsame diode, slightly higher Vf, higher reverse voltage"
-		(exclude_from_sim no)
-		(at 15.24 22.86 0)
-		(effects
-			(font
-				(size 1.27 1.27)
-			)
-			(justify left bottom)
-		)
-	)
 	(text "I2C Isolation"
 		(exclude_from_sim no)
@@
 			)
 		)
-		(property "Value" "PMEG2005CT"
+		(property "Value" "BAT54C"
 			(at 39.37 41.91 0)
 			(show_name no)
@@
 			)
 		)
-		(property "Value" "PMEG2005CT"
+		(property "Value" "BAT54C"
 			(at 123.19 114.3 0)
 			(show_name no)
@@
 			)
 		)
-		(property "Value" "PMEG2005CT"
+		(property "Value" "BAT54C"
 			(at 146.05 97.79 0)
 			(show_name no)
@@
 			)
 		)
-		(property "Value" "PMEG2005CT"
+		(property "Value" "BAT54C"
 			(at 170.18 113.03 0)
 			(show_name no)
@@
 			)
 		)
-		(property "Value" "PMEG2005CT"
+		(property "Value" "BAT54C"
 			(at 74.93 22.86 0)
 			(show_name no)
